File: ai03-pcb-guide.sch (KiCad schematic (older format))
At the start: 24 parts, among them SW1 SW_Push, U1 ATmega32U4-AU, Y1 16MHz

Commit message: finish schematic
Parts:
- removed USB1: Molex-0548190589, random-keyboard-parts:Molex-0548190589, symbol random-keyboard-parts:Molex-0548190589
- added R? (x2): 5k, Resistor_SMD:R_0805_2012Metric, symbol Device:R_Small
- added R? (x2): 22, Resistor_SMD:R_0805_2012Metric, symbol Device:R_Small
- added U?: PRTR5V0U2X, symbol random-keyboard-parts:PRTR5V0U2X
- added USB?: HRO-TYPE-C-31-M-12, symbol Type-C:HRO-TYPE-C-31-M-12
Connections:
- net D+: now also R?.1
- net D-: now also R?.1
- net GND: now also R?.2, R?.2, U?.1 (GND), USB?.1 (GND), USB?.12 (GND), USB?.13 (SHIELD)
- net VCC: now also U?.4 (VCC), USB?.11 (VBUS), USB?.2 (VBUS)
- new net: R?.1, USB?.10 (CC2)
- new net: R?.1, USB?.4 (CC1)
- new net: R?.2, U?.3 (IO2), USB?.5 (DN2), USB?.7 (DN1)
- new net: R?.2, U?.2 (IO1), USB?.6 (DP1), USB?.8 (DP2)
- no-connect marks 0 -> 24
Other:
- moved on the sheet: C1, C2, C3, C4, C5, C6, C7, R1, R2, R3, R4, SW1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
